File: hardware/UFC/UFC.kicad_pcb (KiCad board)
At the start: 2 copper layers, 146 x 50 mm, 117 parts, among them J1 KF2510_02, J10 KF2510_02, J11 KF2510_02, J12 KF2510_02, J13 KF2510_02, J14 KF2510_02, J15 KF2510_02, J16 KF2510_02, J17 KF2510_02, J18 KF2510_02, J19 KF2510_02, J2 KF2510_02, J20 KF2510_02, J21 KF2510_02, J22 KF2510_04, J23 KF2510_04, J24 KF2510_04, J25 KF2510_02, J26 KF2510_02, J27 KF2510_04, J28 KF2510_04, J29 KF2510_04, J3 KF2510_02, J30 KF2510_04, J31 Conn_01x02, J32 Conn_01x02, J4 KF2510_02, J5 KF2510_02, J6 KF2510_02, J7 KF2510_02, J8 KF2510_02, J9 KF2510_02, Q1 Q_PMOS_GSD, Q2 Q_PMOS_GSD, U1 74LS00, U2 6N136, U3 6N136

Commit message: Board rev. 1: connect LCD pin 5 (R/W) to GND
On rev. 0 the pin was connected to +5V, the display stayed in read mode.
The fabrication files of rev. 0 are kept in Gerber/rev00, the README lists
the revisions and the rework for existing boards.

Co-Authored-By: Claude Opus 5.5 <noreply@anthropic.com>
Connections:
- DISP1 pad 10: Net-(DISP1-Pad10) -> unconnected-(DISP1-DB3-Pad10)
- DISP1 pad 5: +5V -> GND
- DISP1 pad 7: Net-(DISP1-Pad7) -> unconnected-(DISP1-DB0-Pad7)
- DISP1 pad 8: Net-(DISP1-Pad8) -> unconnected-(DISP1-DB1-Pad8)
- DISP1 pad 9: Net-(DISP1-Pad9) -> unconnected-(DISP1-DB2-Pad9)
- J22 pad 1: Net-(J22-Pad1) -> unconnected-(J22-Pin_1-Pad1)
- J23 pad 1: Net-(J23-Pad1) -> unconnected-(J23-Pin_1-Pad1)
- J24 pad 1: Net-(J24-Pad1) -> unconnected-(J24-Pin_1-Pad1)
- J27 pad 1: Net-(J27-Pad1) -> unconnected-(J27-Pin_1-Pad1)
- J28 pad 1: Net-(J28-Pad1) -> unconnected-(J28-Pin_1-Pad1)
- J29 pad 1: Net-(J29-Pad1) -> unconnected-(J29-Pin_1-Pad1)
- J30 pad 1: Net-(J30-Pad1) -> unconnected-(J30-Pin_1-Pad1)
- MD1 pad 10: Net-(MD1-Pad10) -> unconnected-(MD1A-RST-Pad10)
- MD1 pad 11: Net-(MD1-Pad11) -> unconnected-(MD1B-RX-Pad11)
- MD1 pad 12: Net-(MD1-Pad12) -> unconnected-(MD1B-TX-Pad12)
- MD1 pad 13: Net-(MD1-Pad13) -> unconnected-(MD1B-D2-Pad13)
- MD1 pad 14: Net-(MD1-Pad14) -> unconnected-(MD1B-D3-Pad14)
- MD1 pad 15: Net-(MD1-Pad15) -> unconnected-(MD1B-D4-Pad15)
- MD1 pad 19: Net-(MD1-Pad19) -> unconnected-(MD1B-D8-Pad19)
- MD1 pad 21: Net-(MD1-Pad21) -> unconnected-(MD1B-D10-Pad21)
- MD1 pad 25: Net-(MD1-Pad25) -> unconnected-(MD1B-D14-Pad25)
- MD1 pad 31: Net-(MD1-Pad31) -> unconnected-(MD1B-D20-Pad31)
- MD1 pad 36: Net-(MD1-Pad36) -> unconnected-(MD1B-D25-Pad36)
- MD1 pad 37: Net-(MD1-Pad37) -> unconnected-(MD1B-D26-Pad37)
- MD1 pad 38: Net-(MD1-Pad38) -> unconnected-(MD1B-D27-Pad38)
- MD1 pad 39: Net-(MD1-Pad39) -> unconnected-(MD1B-D28-Pad39)
- MD1 pad 40: Net-(MD1-Pad40) -> unconnected-(MD1B-D29-Pad40)
- MD1 pad 41: Net-(MD1-Pad41) -> unconnected-(MD1B-D30-Pad41)
- MD1 pad 42: Net-(MD1-Pad42) -> unconnected-(MD1B-D31-Pad42)
- MD1 pad 45: Net-(MD1-Pad45) -> unconnected-(MD1C-A2-Pad45)
- MD1 pad 46: Net-(MD1-Pad46) -> unconnected-(MD1C-A3-Pad46)
- MD1 pad 47: Net-(MD1-Pad47) -> unconnected-(MD1C-A4-Pad47)
- MD1 pad 48: Net-(MD1-Pad48) -> unconnected-(MD1C-A5-Pad48)
- MD1 pad 49: Net-(MD1-Pad49) -> unconnected-(MD1C-A6-Pad49)
- MD1 pad 50: Net-(MD1-Pad50) -> unconnected-(MD1C-A7-Pad50)
- MD1 pad 51: Net-(MD1-Pad51) -> unconnected-(MD1C-A8-Pad51)
- MD1 pad 52: Net-(MD1-Pad52) -> unconnected-(MD1C-A9-Pad52)
- MD1 pad 53: Net-(MD1-Pad53) -> unconnected-(MD1C-A10-Pad53)
- MD1 pad 54: Net-(MD1-Pad54) -> unconnected-(MD1C-A11-Pad54)
- MD1 pad 55: Net-(MD1-Pad55) -> unconnected-(MD1C-A12-Pad55)
- MD1 pad 56: Net-(MD1-Pad56) -> unconnected-(MD1C-A13-Pad56)
- MD1 pad 57: Net-(MD1-Pad57) -> unconnected-(MD1C-A14-Pad57)
- MD1 pad 58: Net-(MD1-Pad58) -> unconnected-(MD1C-A15-Pad58)
- MD1 pad 59: Net-(MD1-Pad59) -> unconnected-(MD1C-D32-Pad59)
- U2 pad 1: Net-(U2-Pad1) -> unconnected-(U2-NC-Pad1)
- U2 pad 4: Net-(U2-Pad4) -> unconnected-(U2-NC-Pad4)
- U3 pad 1: Net-(U3-Pad1) -> unconnected-(U3-NC-Pad1)
- U3 pad 4: Net-(U3-Pad4) -> unconnected-(U3-NC-Pad4)
Routing:
- net +5V: track 319.8 -> 316.9 mm
- net GND: track 12.8 -> 12.9 mm, vias 0 -> 29
- net (no net): vias 29 -> 0
Other:
- board text added: "UFC rev. 1 - 12/10/26"
- board text removed: "UFC rev. 0 - 05/10/18"
